Commit message: Update vimalram.xacro

File: vimal_urdf/vimalram_description/urdf/vimalram.xacro (robot description, xacro)
@@ -1,4 +1,4 @@
 <?xml version="1.0" ?>
-<robot name="BRICKS" xmlns:xacro="http://www.ros.org/wiki/xacro">
+<robot name="vimalram" xmlns:xacro="http://www.ros.org/wiki/xacro">
 <xacro:include filename="$(find BRICKS_description)/urdf/materials.xacro" />
 <xacro:include filename="$(find BRICKS_description)/urdf/BRICKS.trans" />
@@ -94,5 +94,5 @@
   <parent link="base_link"/>
   <child link="whell_1"/>
-  <axis xyz="-0.0 -1.0 -0.0"/>
+  <axis xyz="0.0 1.0 0.0"/>
 </joint>
 <joint name="Rigid6" type="fixed">

Commit message: Update vimalram.xacro

File: vimal_urdf/vimalram_description/urdf/vimalram.xacro (robot description, xacro)
@@ -1,7 +1,7 @@
 <?xml version="1.0" ?>
 <robot name="vimalram" xmlns:xacro="http://www.ros.org/wiki/xacro">
-<xacro:include filename="$(find BRICKS_description)/urdf/materials.xacro" />
-<xacro:include filename="$(find BRICKS_description)/urdf/BRICKS.trans" />
-<xacro:include filename="$(find BRICKS_description)/urdf/BRICKS.gazebo" />
+<xacro:include filename="$(find vimalram_description)/urdf/materials.xacro" />
+<xacro:include filename="$(find vimalram_description)/urdf/vimalram.trans" />
+<xacro:include filename="$(find vimalram_description)/urdf/vimalram.gazebo" />
 <link name="base_link">
   <inertial>
@@ -13,5 +13,5 @@
     <origin xyz="0 0 0" rpy="0 0 0"/>
     <geometry>
-      <mesh filename="package://BRICKS_description/meshes/base_link.stl" scale="0.001 0.001 0.001"/>
+      <mesh filename="package://vimalram_description/meshes/base_link.stl" scale="0.001 0.001 0.001"/>
     </geometry>
     <material name="silver"/>
@@ -20,5 +20,5 @@
     <origin xyz="0 0 0" rpy="0 0 0"/>
     <geometry>
-      <mesh filename="package://BRICKS_description/meshes/base_link.stl" scale="0.001 0.001 0.001"/>
+      <mesh filename="package://vimalram_description/meshes/base_link.stl" scale="0.001 0.001 0.001"/>
     </geometry>
   </collision>
@@ -33,5 +33,5 @@
     <origin xyz="0.070143 -0.057368 -0.050083" rpy="0 0 0"/>
     <geometry>
-      <mesh filename="package://BRICKS_description/meshes/whell_2_1.stl" scale="0.001 0.001 0.001"/>
+      <mesh filename="package://vimalram_description/meshes/whell_2_1.stl" scale="0.001 0.001 0.001"/>
     </geometry>
     <material name="silver"/>
@@ -40,5 +40,5 @@
     <origin xyz="0.070143 -0.057368 -0.050083" rpy="0 0 0"/>
     <geometry>
-      <mesh filename="package://BRICKS_description/meshes/whell_2_1.stl" scale="0.001 0.001 0.001"/>
+      <mesh filename="package://vimalram_description/meshes/whell_2_1.stl" scale="0.001 0.001 0.001"/>
     </geometry>
   </collision>
@@ -53,5 +53,5 @@
     <origin xyz="0.070143 0.052632 -0.050083" rpy="0 0 0"/>
     <geometry>
-      <mesh filename="package://BRICKS_description/meshes/whell_1.stl" scale="0.001 0.001 0.001"/>
+      <mesh filename="package://vimalram_description/meshes/whell_1.stl" scale="0.001 0.001 0.001"/>
     </geometry>
     <material name="silver"/>
@@ -60,5 +60,5 @@
     <origin xyz="0.070143 0.052632 -0.050083" rpy="0 0 0"/>
     <geometry>
-      <mesh filename="package://BRICKS_description/meshes/whell_1.stl" scale="0.001 0.001 0.001"/>
+      <mesh filename="package://vimalram_description/meshes/whell_1.stl" scale="0.001 0.001 0.001"/>
     </geometry>
   </collision>
@@ -73,5 +73,5 @@
     <origin xyz="-0.093072 -0.002368 -0.074905" rpy="0 0 0"/>
     <geometry>
-      <mesh filename="package://BRICKS_description/meshes/lidar_1.stl" scale="0.001 0.001 0.001"/>
+      <mesh filename="package://vimalram_description/meshes/lidar_1.stl" scale="0.001 0.001 0.001"/>
     </geometry>
     <material name="silver"/>
@@ -80,5 +80,5 @@
     <origin xyz="-0.093072 -0.002368 -0.074905" rpy="0 0 0"/>
     <geometry>
-      <mesh filename="package://BRICKS_description/meshes/lidar_1.stl" scale="0.001 0.001 0.001"/>
+      <mesh filename="package://vimalram_description/meshes/lidar_1.stl" scale="0.001 0.001 0.001"/>
     </geometry>
   </collision>
